File: eagle/ALMOST4ALLMINI.brd (EAGLE design)
At the start: 40.3 x 49.8 mm, 39 parts, among them IC1 MCP1700-3302E, IC2 ATSHA204A-STUCZ-T, IC3 W25X40CLSNIG, M1 ARDUINO-PRO-MINI, M2 WIRELESS-NRF24L01

Commit message: 56K values IR-Send corrected
Parts:
- added R15: 100, SparkFun-Passives:0805
- added SJ2: NO, SparkFun-Retired:SJ_2S-NO
- C3: value 4.7uf -> 4.7uF; device SparkFun-Passives:0805 -> SparkFun-Capacitors:CPOL-RADIAL-10UF-25V
- R4, R8: value 56k -> 4K7
- R7: value 56k -> 150
- moved C3 0.32 mm to (33.0, 3.17), flipped to the top
- moved R3 0.32 mm to (4.76, 34.9)
Connections:
- new net D3I: JP5.1, R15.2, R3.1, SJ2.1
- net D3: now also R15.1, SJ2.2; no longer JP5.1, R3.1
Routing:
- net D3I: track 0.00 -> 7.98 mm
- net D3: track 15.8 -> 10.4 mm
- net GND: track 59.4 -> 60.7 mm
Other:
- board text added: "ALMOST4ALLMINI Rev. 1.1 By joseraj"
- board text added: "CC-BY-SA"
- board text added: "R15"
- board text added: "SJ2"
- board text removed: "ALMOST4ALLMINI Rev. 1.0 By joseraj"
